File: ESP8266_12F_BASIC.kicad_pcb (KiCad board)
At the start: 2 copper layers, 64.7 x 63.5 mm, 35 parts, among them J1 Conn_01x02_Male, J2 Conn_01x04_Male, Q1 BC547, U1 ESP-12F, U2 AP1117-33

Commit message: major fixes
Parts:
- added G***: LOGO, COSTUMFOOTPRINTS:sneakyTom, F.Cu at (134.9, 106.7)
- added J3: Conn_01x05_Female, Connector_PinHeader_2.54mm:PinHeader_1x05_P2.54mm_Vertical, F.Cu at (157.0, 111.5)
- added R2: 220k, Resistor_SMD:R_0805_2012Metric_Pad1.20x1.40mm_HandSolder, F.Cu at (123.7, 105.9)
- moved TP4 13.7 mm to (128.5, 93.2)
- moved TP6 12.4 mm to (129.3, 88.6)
- moved TP5 6.07 mm to (130.3, 82.5)
- moved BZ1 3.43 mm to (175.9, 101.2)
- moved R1 1.37 mm to (123.7, 102.0)
Connections:
- R1 pad 1: VCC_3V3 -> ESP_ADC
- R1 pad 2: ESP_ADC -> GND
- U1 pad 17: unconnected-(U1-Pad17) -> GPIO2
- U1 pad 21: unconnected-(U1-Pad21) -> GPIO3
- U1 pad 22: unconnected-(U1-Pad22) -> GPIO1
- U1 pad 4: unconnected-(U1-Pad4) -> GPIO16
- U1 pad 5: unconnected-(U1-Pad5) -> GPIO14
Routing:
- net GPIO3: track 0.00 -> 41.7 mm, vias 0 -> 1
- net GPIO1: track 0.00 -> 38.7 mm, vias 0 -> 1
- net GPIO14: track 0.00 -> 32.2 mm, vias 0 -> 1
- net GPIO16: track 0.00 -> 31.6 mm, vias 0 -> 1
- net GPIO2: track 0.00 -> 31.0 mm, vias 0 -> 1
- net ESP_ADC: track 34.6 -> 42.1 mm
- net VCC_3V3: track 127.0 -> 123.2 mm
- net GND: track 0.00 -> 3.21 mm, vias 44 -> 19
- net ESP_EN: track 25.7 -> 22.6 mm
- net Net-(BZ1-Pad1): track 7.78 -> 10.8 mm
- net VCC_IN: track 96.8 -> 98.8 mm
Other:
- board text added: "G1"
- board text added: "G14"
- board text added: "G16"
- board text added: "G2"
- board text added: "G3"
- board text added: "github.com/wytr"

Commit message: caps added and move also added new picture
Parts:
- added C4: 100nF, Capacitor_SMD:C_1206_3216Metric_Pad1.33x1.80mm_HandSolder, F.Cu at (139.2, 98.8)
- moved C3 33.7 mm to (137.6, 91.7), turned to 180 degrees
- moved G*** 4.79 mm to (137.4, 110.7), turned to 30 degrees
Routing:
- net VCC_3V3: track 123.2 -> 127.8 mm, vias 4 -> 6
- net D1_IN: track 36.8 -> 35.5 mm

Commit message: updated gerber
Other:
- board text added: "INPUT"
- board text added: "MH-Z19"
Changed lines of the file:
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@@
     (property "Sheetname" "")
     (attr through_hole)
-    (fp_text reference "J1" (at 1.25 3.55) (layer "B.SilkS")
+    (fp_text reference "J1" (at 1.25 3.556 180) (layer "B.SilkS") hide
       (effects (font (size 1 1) (thickness 0.15)) (justify mirror))
     )
@@
     (property "Sheetname" "")
     (attr through_hole)
-    (fp_text reference "J2" (at 3.75 3.55) (layer "B.SilkS")
+    (fp_text reference "J2" (at 3.937 3.55 180) (layer "B.SilkS") hide
       (effects (font (size 1 1) (thickness 0.15)) (justify mirror))
     )
@@
     (effects (font (size 1 1) (thickness 0.15)))
   )
+  (gr_text "MH-Z19" (at 146.558 127.508) (layer "B.Mask")
+    (effects (font (size 2 2) (thickness 0.25)) (justify mirror))
+  )
+  (gr_text "INPUT" (at 160.401 127.508) (layer "B.Mask")
+    (effects (font (size 2 2) (thickness 0.25)) (justify mirror))
+  )
   (target plus (at 152.4 101.6) (size 5) (width 0.1) (layer "Edge.Cuts"))
   (segment (start 175.895 103.865) (end 170.18 109.58) (width 0.5) (layer "F.Cu") (net 1))
@@
   (via (at 148.082 101.6) (size 0.8) (drill 0.4) (layers "F.Cu" "B.Cu") (free) (net 2))
   (via (at 167.64 121.92) (size 0.8) (drill 0.4) (layers "F.Cu" "B.Cu") (free) (net 2))
-  (via (at 132.08 121.92) (size 0.8) (drill 0.4) (layers "F.Cu" "B.Cu") (free) (net 2))
+  (via (at 129.286 120.396) (size 0.8) (drill 0.4) (layers "F.Cu" "B.Cu") (free) (net 2))
   (segment (start 160.655 94.615) (end 155.335 94.615) (width 0.5) (layer "F.Cu") (net 3))
   (segment (start 161.29 96.7525) (end 161.29 95.25) (width 0.5) (layer "F.Cu") (net 3))
@@
   (segment (start 160.2525 118.6395) (end 160.2525 124.46) (width 0.5) (layer "F.Cu") (net 3))
   (segment (start 167.64 106.045) (end 165.3325 103.7375) (width 0.5) (layer "F.Cu") (net 3))
+  (segment (start 138.43 122.682) (end 142.748 127) (width 0.5) (layer "F.Cu") (net 4))
+  (segment (start 135.763 122.555) (end 123.698 110.49) (width 0.5) (layer "F.Cu") (net 4))
   (segment (start 140.335 83.82) (end 140.335 82.28) (width 0.5) (layer "F.Cu") (net 4))
+  (segment (start 123.698 110.49) (end 123.698 106.918) (width 0.5) (layer "F.Cu") (net 4))
   (segment (start 145.796 89.662) (end 147.828 87.63) (width 0.5) (layer "F.Cu") (net 4))
+  (segment (start 138.43 122.555) (end 135.763 122.555) (width 0.5) (layer "F.Cu") (net 4))
   (segment (start 140.335 82.28) (end 139.97 81.915) (width 0.5) (layer "F.Cu") (net 4))
   (segment (start 138.43 75.565) (end 139.97 75.565) (width 0.5) (layer "F.Cu") (net 4))
   (segment (start 137.6295 98.806) (end 137.6295 96.8125) (width 0.5) (layer "F.Cu") (net 4))
-  (segment (start 151.155 127) (end 144.145 127) (width 0.5) (layer "F.Cu") (net 4))
   (segment (start 160.2525 127) (end 157.455 127) (width 0.5) (layer "F.Cu") (net 4))
-  (segment (start 135.763 122.555) (end 123.698 110.49) (width 0.5) (layer "F.Cu") (net 4))
-  (segment (start 123.698 110.49) (end 123.698 106.918) (width 0.5) (layer "F.Cu") (net 4))
   (segment (start 144.8 89.875) (end 145.013 89.662) (width 0.5) (layer "F.Cu") (net 4))
   (segment (start 158.300489 86.925489) (end 162.359511 86.925489) (width 0.5) (layer "F.Cu") (net 4))
@@
   (segment (start 144.8 89.875) (end 143.215 89.875) (width 0.5) (layer "F.Cu") (net 4))
   (segment (start 143.215 89.875) (end 142.875 89.535) (width 0.5) (layer "F.Cu") (net 4))
+  (segment (start 142.748 127) (end 151.155 127) (width 0.5) (layer "F.Cu") (net 4))
   (segment (start 157.595978 87.63) (end 158.300489 86.925489) (width 0.5) (layer "F.Cu") (net 4))
   (segment (start 162.359511 86.925489) (end 163.195 86.09) (width 0.5) (layer "F.Cu") (net 4))
   (segment (start 145.013 89.662) (end 145.796 89.662) (width 0.5) (layer "F.Cu") (net 4))
-  (segment (start 144.145 127) (end 139.7 122.555) (width 0.5) (layer "F.Cu") (net 4))
   (segment (start 137.795 76.835) (end 137.795 76.2) (width 0.5) (layer "F.Cu") (net 4))
   (segment (start 137.668 98.8445) (end 137.6295 98.806) (width 0.5) (layer "F.Cu") (net 4))
   (segment (start 137.668 100.838) (end 137.668 98.8445) (width 0.5) (layer "F.Cu") (net 4))
   (segment (start 157.455 127) (end 151.155 127) (width 0.5) (layer "F.Cu") (net 4))
+  (segment (start 138.43 122.555) (end 138.43 122.682) (width 0.5) (layer "F.Cu") (net 4))
   (segment (start 137.795 76.2) (end 138.43 75.565) (width 0.5) (layer "F.Cu") (net 4))
-  (segment (start 139.7 122.555) (end 135.763 122.555) (width 0.5) (layer "F.Cu") (net 4))
   (segment (start 147.828 87.63) (end 157.595978 87.63) (width 0.5) (layer "F.Cu") (net 4))
   (via (at 137.668 96.774) (size 0.8) (drill 0.4) (layers "F.Cu" "B.Cu") (net 4))
@@
   (via (at 137.668 100.838) (size 0.8) (drill 0.4) (layers "F.Cu" "B.Cu") (net 4))
   (via (at 137.795 76.835) (size 0.8) (drill 0.4) (layers "F.Cu" "B.Cu") (net 4))
-  (via (at 139.7 122.555) (size 0.8) (drill 0.4) (layers "F.Cu" "B.Cu") (net 4))
+  (via (at 138.43 122.555) (size 0.8) (drill 0.4) (layers "F.Cu" "B.Cu") (net 4))
   (via (at 140.335 83.82) (size 0.8) (drill 0.4) (layers "F.Cu" "B.Cu") (net 4))
-  (segment (start 138.624521 116.605349) (end 138.624521 118.344651) (width 0.5) (layer "B.Cu") (net 4))
   (segment (start 137.580379 91.694) (end 137.668 91.781621) (width 0.5) (layer "B.Cu") (net 4))
+  (segment (start 140.208 107.569) (end 137.668 105.029) (width 0.5) (layer "B.Cu") (net 4))
   (segment (start 137.795 81.28) (end 137.795 76.835) (width 0.5) (layer "B.Cu") (net 4))
-  (segment (start 137.668 115.648828) (end 138.624521 116.605349) (width 0.5) (layer "B.Cu") (net 4))
+  (segment (start 138.43 122.555) (end 140.208 120.777) (width 0.5) (layer "B.Cu") (net 4))
+  (segment (start 137.668 105.029) (end 137.668 100.838) (width 0.5) (layer "B.Cu") (net 4))
+  (segment (start 140.208 120.777) (end 140.208 107.569) (width 0.5) (layer "B.Cu") (net 4))
   (segment (start 137.668 96.774) (end 137.580379 96.686379) (width 0.5) (layer "B.Cu") (net 4))
-  (segment (start 137.668 120.523) (end 139.7 122.555) (width 0.5) (layer "B.Cu") (net 4))
   (segment (start 142.875 89.535) (end 142.875 86.36) (width 0.5) (layer "B.Cu") (net 4))
   (segment (start 140.335 83.82) (end 137.795 81.28) (width 0.5) (layer "B.Cu") (net 4))
-  (segment (start 137.668 119.301172) (end 137.668 120.523) (width 0.5) (layer "B.Cu") (net 4))
   (segment (start 137.580379 96.686379) (end 137.580379 91.694) (width 0.5) (layer "B.Cu") (net 4))
   (segment (start 142.875 86.36) (end 140.335 83.82) (width 0.5) (layer "B.Cu") (net 4))
   (segment (start 140.716 91.694) (end 137.580379 91.694) (width 0.5) (layer "B.Cu") (net 4))
-  (segment (start 137.668 100.838) (end 137.668 115.648828) (width 0.5) (layer "B.Cu") (net 4))
   (segment (start 142.875 89.535) (end 140.716 91.694) (width 0.5) (layer "B.Cu") (net 4))
-  (segment (start 138.624521 118.344651) (end 137.668 119.301172) (width 0.5) (layer "B.Cu") (net 4))
   (segment (start 146.14 99.39) (end 147.625 99.39) (width 0.5) (layer "F.Cu") (net 5))
   (segment (start 154.94 98.425) (end 157.175 96.19) (width 0.5) (layer "F.Cu") (net 5))
