File: ESP8266_12F_BASIC.kicad_pcb (KiCad board)
At the start: 2 copper layers, 64.7 x 63.5 mm, 39 parts, among them J1 Conn_01x02_Male, J2 Conn_01x04_Male, J3 Conn_01x05_Female, Q1 BC547, U1 ESP-12F, U2 AP1117-33

Commit message: reset
Parts:
- added R8: 10k, Resistor_SMD:R_0805_2012Metric_Pad1.20x1.40mm_HandSolder, F.Cu at (161.8, 85.7)
- added TP8: TestPoint, TestPoint:TestPoint_THTPad_D3.0mm_Drill1.5mm, F.Cu at (130.0, 112.0)
- moved TP3 3.56 mm to (166.4, 96.9)
- moved R6 1.15 mm to (163.1, 90.0)
- moved R2 0.76 mm to (140.2, 78.1)
- moved R3 0.76 mm to (140.2, 75.6)
- moved U1 0.76 mm to (151.6, 79.4)
- moved R5 0.65 mm to (163.8, 85.0)
- moved R4 0.51 mm to (140.5, 81.9)
Connections:
- J3 pad 2: GPIO2 -> unconnected-(J3-Pad2)
- U1 pad 17: GPIO2 -> Net-(R8-Pad2)
Routing:
- net GPIO2: track 31.0 -> 0.00 mm, vias 1 -> 0
- net VCC_3V3: track 128.0 -> 132.1 mm
- net Net-(R8-Pad2): track 0.00 -> 3.04 mm
- net Net-(R5-Pad2): track 3.28 -> 5.57 mm
- net GND: track 3.21 -> 4.35 mm
- net Net-(R6-Pad2): track 3.21 -> 4.31 mm
- net ESP_ADC: track 42.3 -> 41.5 mm
Other:
- board text removed: "G2"

Commit message: old state no hotfix
Parts:
- removed R8: 10k, Resistor_SMD:R_0805_2012Metric_Pad1.20x1.40mm_HandSolder
- removed TP8: TestPoint, TestPoint:TestPoint_THTPad_D3.0mm_Drill1.5mm
- moved TP3 3.56 mm to (166.4, 93.3)
- moved R6 1.15 mm to (163.2, 88.9)
- moved R2 0.76 mm to (141.0, 78.1)
- moved R3 0.76 mm to (141.0, 75.6)
- moved U1 0.76 mm to (152.4, 79.4)
- moved R5 0.65 mm to (163.2, 85.1)
- moved R4 0.51 mm to (141.0, 81.9)
Connections:
- J3 pad 2: unconnected-(J3-Pad2) -> GPIO2
- U1 pad 17: Net-(R8-Pad2) -> GPIO2
Routing:
- net GPIO2: track 0.00 -> 31.0 mm, vias 0 -> 1
- net VCC_3V3: track 132.1 -> 128.0 mm
- net Net-(R8-Pad2): track 3.04 -> 0.00 mm
- net Net-(R5-Pad2): track 5.57 -> 3.28 mm
- net GND: track 4.35 -> 3.21 mm
- net Net-(R6-Pad2): track 4.31 -> 3.21 mm
- net ESP_ADC: track 41.5 -> 42.3 mm
Other:
- board text added: "G2"

Commit message: hotfix
Parts:
- added R8: 10k, Resistor_SMD:R_0805_2012Metric_Pad1.20x1.40mm_HandSolder, F.Cu at (161.8, 85.7)
- moved TP3 3.56 mm to (166.4, 96.9)
- moved R6 1.15 mm to (163.1, 90.0)
- moved R2 0.76 mm to (140.2, 78.1)
- moved R3 0.76 mm to (140.2, 75.6)
- moved U1 0.76 mm to (151.6, 79.4)
- moved R5 0.65 mm to (163.8, 85.0)
- moved R4 0.51 mm to (140.5, 81.9)
Connections:
- J3 pad 2: GPIO2 -> unconnected-(J3-Pad2)
- U1 pad 17: GPIO2 -> Net-(R8-Pad2)
Routing:
- net GPIO2: track 31.0 -> 0.00 mm, vias 1 -> 0
- net BUZZ: track 39.0 -> 35.6 mm
- net Net-(R8-Pad2): track 0.00 -> 3.04 mm
- net Net-(R5-Pad2): track 3.28 -> 5.57 mm
- net GND: track 3.21 -> 4.35 mm
- net Net-(R6-Pad2): track 3.21 -> 4.31 mm
- net ESP_ADC: track 42.3 -> 41.5 mm
Other:
- board text removed: "G2"

Commit message: weird shit
Parts:
- removed R8: 10k, Resistor_SMD:R_0805_2012Metric_Pad1.20x1.40mm_HandSolder
- moved TP3 3.56 mm to (166.4, 93.3)
- moved R6 1.15 mm to (163.2, 88.9)
- moved R2 0.76 mm to (141.0, 78.1)
- moved R3 0.76 mm to (141.0, 75.6)
- moved U1 0.76 mm to (152.4, 79.4)
- moved R5 0.65 mm to (163.2, 85.1)
- moved R4 0.51 mm to (141.0, 81.9)
Connections:
- J3 pad 2: unconnected-(J3-Pad2) -> GPIO2
- U1 pad 17: Net-(R8-Pad2) -> GPIO2
Routing:
- net GPIO2: track 0.00 -> 31.0 mm, vias 0 -> 1
- net BUZZ: track 35.6 -> 39.0 mm
- net Net-(R8-Pad2): track 3.04 -> 0.00 mm
- net Net-(R5-Pad2): track 5.57 -> 3.28 mm
- net GND: track 4.35 -> 3.21 mm
- net Net-(R6-Pad2): track 4.31 -> 3.21 mm
- net ESP_ADC: track 41.5 -> 42.3 mm
Other:
- board text added: "G2"
