File: ESP8266_12F_BASIC.kicad_sch (KiCad schematic)
At the start: 37 parts, among them J1 Conn_01x02_Male, J2 Conn_01x04_Male, J3 Conn_01x05_Female, Q1 BC547, U1 ESP-12F, U2 AP1117-33

Commit message: hotfix
Parts:
- added R8: 10k, Resistor_SMD:R_0805_2012Metric_Pad1.20x1.40mm_HandSolder, symbol Device:R_Small
Connections:
- net VCC_3V3: now also R8.1
- net GPIO2: no longer names the net of J3.2 (Pin_2)
- net GPIO2: no longer U1.17 (GPIO2)
- new net: R8.2, U1.17 (GPIO2)
- no-connect marks 7 -> 8
Other:
- note added: "floating"
- note added: "high running"
- moved on the sheet: C3, C4, J2
